File: michele58_choc_spacing_hs-flip/michele58.kicad_pcb (KiCad board)
At the start: 2 copper layers, 145.1 x 108 mm, 103 parts, among them J1 OLED, J2 i2c, J3 i2c, J4 LED, U1 EliteC_Pro_Micro, U2 TRRS

Commit message: latest changes
Parts:
- D30, D31, D32, D33, D34, D35, D36, D37, D38, D39, D40, D41, D42, D43, D44, D45, D46, D47, D48, D49, D50, D51, D52, D53, D54, D55, D56, D57, D58: value LED_SK6812MINI -> SK6812MINI-E
- moved D8 8.17 mm to (131.6, 64.3), turned to -90 degrees
- moved D28 8.16 mm to (150.1, 115.3), turned to -90 degrees
- moved D15 8.15 mm to (150.1, 80.3), turned to -90 degrees
- moved D10 8.15 mm to (168.6, 64.3), turned to -90 degrees
- moved D16 8.08 mm to (168.6, 81.9), turned to -90 degrees
- moved D26 8.08 mm to (109.1, 119.6), turned to -70 degrees
- moved D14 8.08 mm to (131.6, 81.9), turned to -90 degrees
- moved D24 8.08 mm to (205.6, 108.0), turned to -90 degrees
- moved D27 8.08 mm to (131.6, 116.9), turned to -90 degrees
- moved D7 8.06 mm to (113.0, 66.4), turned to -90 degrees
- moved D29 8.06 mm to (168.6, 116.9), turned to -90 degrees
- moved D12 8.04 mm to (205.6, 73.0), turned to -90 degrees
- moved D13 8.04 mm to (113.1, 83.9), turned to -90 degrees
- moved D23 8.03 mm to (187.1, 108.0), turned to -90 degrees
- moved D9 8.01 mm to (150.1, 63.0), turned to -90 degrees
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Connections:
- D30 pad 1: Net-(D30-DOUT) -> VCC
- D30 pad 2: GND -> Net-(D30-DOUT)
- D30 pad 3: LED -> GND
- D30 pad 4: VCC -> LED
- D31 pad 1: Net-(D31-DOUT) -> VCC
- D31 pad 2: GND -> Net-(D31-DOUT)
- D31 pad 3: Net-(D30-DOUT) -> GND
- D31 pad 4: VCC -> Net-(D31-DIN)
- D32 pad 1: Net-(D32-DOUT) -> VCC
- D32 pad 2: GND -> Net-(D32-DOUT)
- D32 pad 3: Net-(D31-DOUT) -> GND
- D32 pad 4: VCC -> Net-(D31-DOUT)
- D33 pad 1: Net-(D33-DOUT) -> VCC
- D33 pad 2: GND -> Net-(D33-DOUT)
- D33 pad 3: Net-(D32-DOUT) -> GND
- D33 pad 4: VCC -> Net-(D33-DIN)
- D34 pad 1: Net-(D34-DOUT) -> VCC
- D34 pad 2: GND -> Net-(D34-DOUT)
- D34 pad 3: Net-(D33-DOUT) -> GND
- D34 pad 4: VCC -> Net-(D33-DOUT)
- D35 pad 1: Net-(D35-DOUT) -> VCC
- D35 pad 2: GND -> unconnected-(D35-DOUT-Pad2)
- D35 pad 3: Net-(D34-DOUT) -> GND
- D35 pad 4: VCC -> Net-(D35-DIN)
- D36 pad 1: Net-(D36-DOUT) -> VCC
- D36 pad 2: GND -> Net-(D36-DOUT)
- D36 pad 3: Net-(D36-DIN) -> GND
- D36 pad 4: VCC -> Net-(D30-DOUT)
- D37 pad 1: Net-(D36-DIN) -> VCC
- D37 pad 2: GND -> Net-(D31-DIN)
- D37 pad 3: Net-(D37-DIN) -> GND
- D37 pad 4: VCC -> Net-(D37-DIN)
- D38 pad 1: Net-(D37-DIN) -> VCC
- D38 pad 2: GND -> Net-(D38-DOUT)
- D38 pad 3: Net-(D38-DIN) -> GND
- D38 pad 4: VCC -> Net-(D32-DOUT)
- D39 pad 1: Net-(D38-DIN) -> VCC
- D39 pad 2: GND -> Net-(D33-DIN)
- D39 pad 3: Net-(D39-DIN) -> GND
- D39 pad 4: VCC -> Net-(D39-DIN)
- D40 pad 1: Net-(D39-DIN) -> VCC
- D40 pad 2: GND -> Net-(D40-DOUT)
- D40 pad 3: Net-(D40-DIN) -> GND
- D40 pad 4: VCC -> Net-(D34-DOUT)
- D41 pad 1: Net-(D40-DIN) -> VCC
- D41 pad 2: GND -> Net-(D35-DIN)
- D41 pad 3: Net-(D35-DOUT) -> GND
- D41 pad 4: VCC -> Net-(D41-DIN)
- D42 pad 1: Net-(D42-DOUT) -> VCC
- D42 pad 2: GND -> Net-(D42-DOUT)
- D42 pad 3: Net-(D36-DOUT) -> GND
- D42 pad 4: VCC -> Net-(D36-DOUT)
- D43 pad 1: Net-(D43-DOUT) -> VCC
- D43 pad 2: GND -> Net-(D37-DIN)
- D43 pad 3: Net-(D42-DOUT) -> GND
- D43 pad 4: VCC -> Net-(D43-DIN)
- D44 pad 1: Net-(D44-DOUT) -> VCC
- D44 pad 2: GND -> Net-(D44-DOUT)
- D44 pad 3: Net-(D43-DOUT) -> GND
- D44 pad 4: VCC -> Net-(D38-DOUT)
- D45 pad 1: Net-(D45-DOUT) -> VCC
- D45 pad 2: GND -> Net-(D39-DIN)
- D45 pad 3: Net-(D44-DOUT) -> GND
- D45 pad 4: VCC -> Net-(D45-DIN)
- D46 pad 1: Net-(D46-DOUT) -> VCC
- D46 pad 2: GND -> Net-(D46-DOUT)
- D46 pad 3: Net-(D45-DOUT) -> GND
- D46 pad 4: VCC -> Net-(D40-DOUT)
- D47 pad 1: Net-(D47-DOUT) -> VCC
- D47 pad 2: GND -> Net-(D41-DIN)
- D47 pad 3: Net-(D46-DOUT) -> GND
- D47 pad 4: VCC -> Net-(D47-DIN)
- D48 pad 1: Net-(D48-DOUT) -> VCC
- D48 pad 2: GND -> Net-(D48-DOUT)
- D48 pad 3: Net-(D48-DIN) -> GND
- D48 pad 4: VCC -> Net-(D42-DOUT)
- D49 pad 1: Net-(D48-DIN) -> VCC
- D49 pad 2: GND -> Net-(D43-DIN)
- D49 pad 3: Net-(D49-DIN) -> GND
- D49 pad 4: VCC -> Net-(D49-DIN)
- D50 pad 1: Net-(D49-DIN) -> VCC
- D50 pad 2: GND -> Net-(D50-DOUT)
- D50 pad 3: Net-(D50-DIN) -> GND
- D50 pad 4: VCC -> Net-(D44-DOUT)
- D51 pad 1: Net-(D50-DIN) -> VCC
- D51 pad 2: GND -> Net-(D45-DIN)
- D51 pad 3: Net-(D51-DIN) -> GND
- D51 pad 4: VCC -> Net-(D51-DIN)
- D52 pad 1: Net-(D51-DIN) -> VCC
- D52 pad 2: GND -> Net-(D52-DOUT)
- D52 pad 3: Net-(D52-DIN) -> GND
- D52 pad 4: VCC -> Net-(D46-DOUT)
- D53 pad 1: Net-(D52-DIN) -> VCC
- D53 pad 2: GND -> Net-(D47-DIN)
- D53 pad 3: Net-(D47-DOUT) -> GND
- D53 pad 4: VCC -> Net-(D53-DIN)
- D54 pad 1: Net-(D54-DOUT) -> VCC
- D54 pad 2: GND -> Net-(D54-DOUT)
- D54 pad 3: Net-(D48-DOUT) -> GND
- D54 pad 4: VCC -> Net-(D48-DOUT)
- D55 pad 1: Net-(D55-DOUT) -> VCC
- D55 pad 2: GND -> Net-(D49-DIN)
- D55 pad 3: Net-(D54-DOUT) -> GND
- D55 pad 4: VCC -> Net-(D54-DOUT)
- D56 pad 1: Net-(D56-DOUT) -> VCC
- D56 pad 2: GND -> Net-(D56-DOUT)
- D56 pad 3: Net-(D55-DOUT) -> GND
- D56 pad 4: VCC -> Net-(D50-DOUT)
- D57 pad 1: Net-(D57-DOUT) -> VCC
- D57 pad 2: GND -> Net-(D51-DIN)
- D57 pad 3: Net-(D56-DOUT) -> GND
- D57 pad 4: VCC -> Net-(D56-DOUT)
- D58 pad 1: unconnected-(D58-DOUT-Pad1) -> VCC
- D58 pad 2: GND -> Net-(D53-DIN)
- D58 pad 3: Net-(D57-DOUT) -> GND
- D58 pad 4: VCC -> Net-(D52-DOUT)
Routing:
- net GND: track 98.5 -> 900.1 mm, vias 2 -> 31
- net VCC: track 112.1 -> 857.5 mm, vias 1 -> 34
- net Column 4: track 12.2 -> 252.7 mm, vias 0 -> 6
- net Column 3: track 12.5 -> 244.5 mm, vias 0 -> 6
- net Column 5: track 18.6 -> 245.0 mm, vias 1 -> 4
- net Column 2: track 7.93 -> 233.6 mm, vias 0 -> 6
- net Column 1: track 5.83 -> 206.7 mm, vias 0 -> 6
- net Row 4: track 31.4 -> 203.6 mm, vias 1 -> 7
- net Row 3: track 40.5 -> 209.9 mm, vias 1 -> 9
- net Row 0: track 24.5 -> 192.5 mm, vias 0 -> 7
- net Row 2: track 41.3 -> 201.0 mm, vias 1 -> 9
- net Column 0: track 44.6 -> 198.5 mm, vias 4 -> 5
- net Row 1: track 41.5 -> 188.9 mm, vias 1 -> 9
- net Net-(D53-DIN): track 0.00 -> 73.4 mm, vias 0 -> 3
- net Net-(D49-DIN): track 0.00 -> 47.2 mm, vias 0 -> 6
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Other:
- outline, holes or cut-outs redrawn

Commit message: latest changes
Parts:
- added H5: Mounting_Hole, MountingHole:MountingHole_3.2mm_M3, F.Cu at (90.3, 122.3)
- added JP1: Jumper, mylocal_footprints:jumper_data-MOD, B.Cu at (88.7, 74.4)
- added JP2: Jumper, mylocal_footprints:jumper_data-MOD, B.Cu at (86.2, 74.4)
- added JP3: Jumper, mylocal_footprints:jumper_data-MOD, B.Cu at (83.6, 74.4)
- added JP4: Jumper, mylocal_footprints:jumper_data-MOD, B.Cu at (81.1, 74.4)
- added JP6: Jumper, mylocal_footprints:jumper_data-MOD, F.Cu at (81.1, 123.3)
- added JP6: Jumper, mylocal_footprints:jumper_data-MOD, B.Cu at (81.1, 123.3)
- added JP7: Jumper, mylocal_footprints:jumper_data-MOD, F.Cu at (90.3, 118.3)
- added JP7: Jumper, mylocal_footprints:jumper_data-MOD, B.Cu at (90.3, 118.3)
- added Thumbstick1: ~, mylocal_footprints:Mini 2-Axis Analog Thumbstick, F.Cu at (80.5, 111.1)
- U1: value EliteC_Pro_Micro -> Elite-Pi_RP2040; footprint Keebio-Parts:Elite-C -> mylocal_footprints:ProMicro
- U2: footprint ScottoKeebs_Components:TRRS_PJ-320A -> mylocal_footprints:TRRS-PJ-320A-double-sided
- moved H4 144.5 mm to (188.4, 67.5)
- moved H3 134.8 mm to (188.5, 102.5)
- moved H1 111.3 mm to (114.4, 60.9)
- moved H2 69.3 mm to (114.4, 95.9)
- moved JP4 4.05 mm to (88.7, 74.4)
- moved JP1 4.03 mm to (81.1, 74.4)
- moved JP3 4.01 mm to (86.2, 74.4)
- moved JP2 4.01 mm to (83.6, 74.4)
- moved U2 1.00 mm to (70.6, 42.9)
- moved U1 0.69 mm to (85.4, 59.7), turned to 0 degrees
- moved J1 0.12 mm to (81.1, 78.3)
Connections:
- U1 pad 19: unconnected-(U1-A2/PF5-Pad19) -> ThumbY
- U1 pad 20: unconnected-(U1-A3/PF4-Pad20) -> ThumbX
Routing:
- net GND: track 900.1 -> 1027.0 mm, vias 31 -> 35
- net ThumbX: track 0.00 -> 87.9 mm, vias 0 -> 1
- net ThumbY: track 0.00 -> 80.0 mm, vias 0 -> 1
- net VCC: track 857.5 -> 935.7 mm, vias 34 -> 35
- net SDA: track 15.2 -> 44.9 mm, vias 0 -> 4
- net SCL: track 15.6 -> 39.7 mm, vias 1 -> 3
- net Column 5: track 245.0 -> 265.0 mm
- net Column 1: track 206.7 -> 225.8 mm
- net Column 2: track 233.6 -> 252.0 mm, vias 6 -> 8
- net Column 0: track 198.5 -> 216.8 mm
- net Column 3: track 244.5 -> 262.7 mm, vias 6 -> 8
- net DATA: track 27.0 -> 44.9 mm, vias 0 -> 2
- net unconnected-(U1-4/PD4-Pad7): track 0.00 -> 17.0 mm, vias 0 -> 1
- net Column 4: track 252.7 -> 269.4 mm
- net unconnected-(U1-RAW-Pad24): track 0.00 -> 14.5 mm
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Other:
- board size 145.1 x 108 mm -> 143.7 x 108.3 mm

Commit message: more tweaks
Parts:
- added G***: LOGO, mylocal_footprints:vf1-valkyrie, F.Cu at (80.7, 91.4)
- added G***: LOGO, mylocal_footprints:vf1-valkyrie, B.Cu at (80.7, 91.4)
- moved U2 0.22 mm to (70.6, 43.1)
Connections:
- JP1 pad 1: Net-(J1-P1) -> Net-(J1-P4)
- JP2 pad 1: Net-(J1-P2) -> Net-(J1-P3)
- JP3 pad 1: Net-(J1-P3) -> Net-(J1-P2)
- JP4 pad 1: Net-(J1-P4) -> Net-(J1-P1)
- JP6 pad 2: GND -> VCC
- JP7 pad 1: Net-(JP7-A) -> VCC
- JP7 pad 2: VCC -> Net-(JP7-A) (x2)
Routing:
- net Net-(D53-DIN): track 73.3 -> 75.3 mm
- net VCC: track 935.7 -> 934.1 mm
- net GND: track 1027.0 -> 1025.4 mm
Other:
- board size 143.7 x 108.3 mm -> 143.6 x 107.9 mm
- board text added: "VF1 Valyrie v1.0.0-rc1 by Richard Nunez (Antebios)"

Commit message: fixes
Parts:
- moved G*** 1.50 mm to (80.7, 89.9) (x2)
