File: michele58_choc_spacing_hs-flip/pcb/michele58.kicad_sch (KiCad schematic)
At the start: 107 parts, among them J1 OLED, J2 i2c, J3 i2c, J4 LED, U1 Elite-Pi_RP2040, U2 TRRS

Commit message: Made mounting holes larger, added mask, and add STL for bottom case with spacers.
Parts:
- H1, H2, H3, H4, H5: footprint MountingHole:MountingHole_3.2mm_M3 -> MountingHole:MountingHole_3.5mm
Changed lines of the file:
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@@
       (effects (font (size 1.27 1.27)) (justify left))
     )
-    (property "Footprint" "MountingHole:MountingHole_3.2mm_M3" (at 191.008 132.461 0)
+    (property "Footprint" "MountingHole:MountingHole_3.5mm" (at 191.008 132.461 0)
       (effects (font (size 1.27 1.27)) hide)
     )
@@
       (effects (font (size 1.27 1.27)) (justify left))
     )
-    (property "Footprint" "MountingHole:MountingHole_3.2mm_M3" (at 190.627 141.859 0)
+    (property "Footprint" "MountingHole:MountingHole_3.5mm" (at 190.627 141.859 0)
       (effects (font (size 1.27 1.27)) hide)
     )
@@
       (effects (font (size 1.27 1.27)) (justify left))
     )
-    (property "Footprint" "MountingHole:MountingHole_3.2mm_M3" (at 190.881 137.16 0)
+    (property "Footprint" "MountingHole:MountingHole_3.5mm" (at 190.881 137.16 0)
       (effects (font (size 1.27 1.27)) hide)
     )
@@
       (effects (font (size 1.27 1.27)) (justify left))
     )
-    (property "Footprint" "MountingHole:MountingHole_3.2mm_M3" (at 190.881 146.685 0)
+    (property "Footprint" "MountingHole:MountingHole_3.5mm" (at 190.881 146.685 0)
       (effects (font (size 1.27 1.27)) hide)
     )
@@
       (effects (font (size 1.27 1.27)) (justify left))
     )
-    (property "Footprint" "MountingHole:MountingHole_3.2mm_M3" (at 191.135 151.765 0)
-      (effects (font (size 1.27 1.27)) hide)
-    )
+    (property "Footprint" "MountingHole:MountingHole_3.5mm" (at 191.135 151.765 0)
+      (effects (font (size 1.27 1.27)) hide)
+    )
