File: michele42_choc_spacing_wl-flip/pcb/michele42.kicad_sch (KiCad schematic)
At the start: 84 parts, among them J1 Battery, J2 OLED-5Pin, J4 LED, SW1 SW_Power, U1 MCU_Nice_Nano_V2

Commit message: Small fixes and images
Other:
- title: VF2 Valkyrie Choc RGB -> VF-31A Kairos Choc RGB
- moved on the sheet: H1, H2, H3, H4, H5, H6, H7, J1, JP6, JP7, SW1, Thumbstick1
