File: kairos42_choc_spacing_trackpad_wl-flip/pcb/michele42_trackpad.kicad_pcb (KiCad board)
At the start: 2 copper layers, 139.6 x 90.1 mm, 104 parts, among them J1 Battery, J2 OLED-5Pin, J4 LED, SW1 SW_Power, U1 MCU_Nice_Nano_V2

Commit message: Resolve DRC errors
Parts:
- removed GND, SDA, VCC: TestPoint, TestPoint:TestPoint_Pad_D1.0mm
- removed REF** (x2): OSHW-Logo_7.5x8mm_SilkScreen, Symbol:OSHW-Logo_7.5x8mm_SilkScreen
- moved H2 0.85 mm to (135.5, 123.0)
Connections:
- D26 pad 3: Net-(D26-GND) -> GND
- D27 pad 3: Net-(D26-GND) -> GND
- D32 pad 3: Net-(D26-GND) -> GND
- D33 pad 3: Net-(D26-GND) -> GND
- D38 pad 3: Net-(D26-GND) -> GND
- D39 pad 3: Net-(D26-GND) -> GND
Routing:
- net unconnected-(D27-DOUT-Pad2): track 2.96 -> 0.42 mm, vias 1 -> 0
- net GND: track 751.5 -> 752.5 mm
