File: kairos42_choc_spacing_trackpad_wl-flip/pcb/michele42_trackpad-splayed.kicad_sch (KiCad schematic)
At the start: 92 parts, among them J1 Battery, J3 OLED-5Pin, J4 LED, SW1 SW_Power, U1 MCU_Nice_Nano_V2

Commit message: Trackpad cas stuff - wip again
Parts:
- removed D16: SK6812MINI-E, mylocal_footprints:SK6812-MINI-E-double-side, symbol SofleKeyboard1:LED_SK6812MINI-E-alt
- removed D38: Diode, mylocal_footprints:Diode_SOD-123-double-sided, symbol ScottoKeebs:Placeholder_Diode
- removed S16: Keyswitch, mylocal_footprints:Choc_Hotswap-double-sided, symbol ScottoKeebs:Placeholder_Keyswitch
- added JP6, JP7: Jumper, mylocal_footprints:jumper_data-MOD, symbol Jumper:Jumper_2_Open
- added Thumbstick1: (no value), mylocal_footprints:Mini 2-Axis Analog Thumbstick, symbol mylocalSymbols1:Mini_2-Axis_Analog_Thumbstick
- renumbered D23 to D1, D36 to D10, D40 to D11, D43 to D12, D25 to D13, D29 to D14, D33 to D15, D37 to D16, D41 to D17, D44 to D18, D26 to D19, D27 to D2, D30 to D20, D34 to D21, D1 to D22, D5 to D23, D9 to D24, D13 to D25, D17 to D26, D20 to D27, D2 to D28, D6 to D29, D31 to D3, D10 to D30, D14 to D31, D18 to D32, D21 to D33, D3 to D34, D7 to D35, D11 to D36, D15 to D37, D19 to D38, D22 to D39, D35 to D4, D4 to D40, D8 to D41, D12 to D42, D39 to D5, D42 to D6, D24 to D7, D28 to D8, D32 to D9, J3 to J2, J2 to J3, S14 to S10, S18 to S11, S21 to S12, S3 to S13, S7 to S14, S11 to S15, S15 to S16, S19 to S17, S22 to S18, S4 to S19, S5 to S2, S8 to S20, S12 to S21, S9 to S3, S13 to S4, S17 to S5, S20 to S6, S2 to S7, S6 to S8, S10 to S9
Connections:
- net CS: no longer U1.7 (D4)
- net DRDY: now also U1.6 (D3); no longer U1.2 (D0)
- net GND: now also JP6.2 (B), Thumbstick1.1 (GND)
- net LED: now also U1.5 (D2); no longer U1.1 (D1)
- net MOSI: no longer U1.5 (D2)
- net SCK: no longer U1.6 (D3)
- net SCL: now also U1.2 (D0); no longer U1.19 (D20)
- net SDA: now also U1.1 (D1); no longer U1.20 (D21)
- net VCC: now also JP7.2 (B), Thumbstick1.3 (VCC)
- net at D42.2 (DOUT): now also D37.4 (DIN)
- new net: JP7.1 (A), Thumbstick1.4 (VCC)
- new net: JP6.1 (A), Thumbstick1.6 (GND)
- new net ThumbX: Thumbstick1.2 (X), U1.20 (D21)
- new net ThumbY: Thumbstick1.5 (Y), U1.19 (D20)
- no-connect marks 9 -> 3
Other:
- moved on the sheet: D22, D23, D24, D25, D26, D27, D28, D29, D30, D31, D32, D33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
