File: kairos42_choc_spacing_trackpad_wl-flip/case/michele42_trackpad.kicad_pcb (KiCad board)
At the start: 2 copper layers, 135.8 x 90.1 mm, 28 parts

Commit message: Trackpad cas stuff - wip again
Other:
- outline, holes or cut-outs redrawn
Changed lines of the file:
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@@
+	)
+	(gr_line
+		(start 72 56.697749)
+		(end 72 131.5)
+		(stroke
+			(width 0.1)
+			(type dash)
+		)
+		(layer "Edge.Cuts")
+	)
+	(gr_line
+		(start 72 56.697749)
+		(end 96.499936 56.697749)
+		(stroke
+			(width 0.1)
+			(type dash)
+		)
+		(layer "Edge.Cuts")
 	)
 	(gr_line
@@
 		(end 96.5 116.5)
 		(stroke
-			(width 0.2)
-			(type default)
+			(width 0.1)
+			(type solid)
 		)
 		(layer "Edge.Cuts")
@@
 		(stroke
 			(width 0.1)
-			(type default)
+			(type solid)
 		)
 		(layer "Edge.Cuts")
@@
 		(layer "User.2")
 	)
+	(dimension
+		(type orthogonal)
+		(layer "Edge.Cuts")
+		(pts
+			(xy 135.331753 108.015542) (xy 135.331753 94.215542)
+		)
+		(height -0.831753)
+		(orientation 1)
+		(format
+			(prefix "")
+			(suffix "")
+			(units 3)
+			(units_format 1)
+			(precision 4)
+		)
+		(style
+			(thickness 0.2)
+			(arrow_length 1.27)
+			(text_position_mode 0)
+			(arrow_direction outward)
+			(extension_height 0.58642)
+			(extension_offset 0.5)
+			(keep_text_aligned yes)
+		)
+		(gr_text "13.8000 mm"
+			(at 133.35 101.115542 90)
+			(layer "Edge.Cuts")
+			(effects
+				(font
+					(size 1 1)
+					(thickness 0.15)
+				)
+			)
+		)
+	)
 	(group ""
